File: RaspberryPiGamingBoard.sch (EAGLE design)
At the start: 42 parts, among them IC3 TP4056, IC5 PAM8403

Commit message: Batteries and Buttons Rearranged
Parts:
- removed C10: 1u, CEDT_JANUARY_2015_v6:CAP0805
- removed CHRGD, CHRGNG: LED3MM, Arduino_Hackathon_v5:LED3MM
- removed IC3: TP4056, tp4056:TP4056
- removed ON: LED3MM, CEDT:LED3MM
- removed R5: 10K, CEDT_JANUARY_2015_v5:RESISTOR0207/7
- removed R6, R7, R8: 1K, CEDT_JANUARY_2015_v5:RESISTOR0207/7
- removed U$3: USB(POWER), CEDT_JANUARY_2015_v5:USB(POWER)
- added BT2: BK-18650-PC2, BK-18650-PC2:BK-18650-PC2
- added C8: 100u, rcl:CPOL-USE5-10.5
- added CON1: (no value), CEDT_JANUARY_2015_v6:POWER_CON
- C7: value 47u -> 100u; device BeagleBone_Blue_R3:CAPACITOR-PE5-8.5 -> rcl:CPOL-USE5-10.5
- D1: value 1N5819-B -> 1N5819; device diode:1N5819-B -> CEDT_JANUARY_2015_v6:1N5819
- L1: value 33uH -> 100uH
- R3: value 6.8k -> 2.2k; device rcl:R-US_0207/10 -> CEDT_JANUARY_2015_v6:RESISTOR0207/7
- R4: value 2.2k -> 6.8k; device rcl:R-US_0207/10 -> CEDT_JANUARY_2015_v6:RESISTOR0207/7
- VR1: value XL6009 -> LM2576T-ADJ/NOPB; device XL6009:XL6009 -> LM2576T-ADJ_NOPB:LM2576T-ADJ/NOPB
Connections:
- removed net N$15: CHRGD.C, R7.1
- removed net N$16: IC3.CHRG, R6.2
- removed net N$17: IC3.STDBY, R7.2
- removed net N$18: C10.1, C7.+, L1.1, POWER_SWITCH.1, VR1.EN, VR1.VIN
- removed net N$22: ON.A, R8.2
- removed net N$6: IC3.PROG, R5.2
- removed net USB_VCC: CHRGD.A, CHRGNG.A, IC3.CE, IC3.VCC, R8.1, U$3.VCC
- new net BUCK_IN: C7.+, POWER_SWITCH.1, VR1.VIN
- net +5V: now also VR1.FEEDBACK; no longer VR1.FB
- net BATTERY_IN+: now also BT2.+, CON1.+; no longer BT1.+, IC3.BAT
- net GND: now also C8.-, CON1.-, CON1.C, D1.A, R3.1, VR1.!ON!/OFF, VR1.GROUND; no longer C10.2, IC3.GND, IC3.TEMP, ON.C, R4.2, R5.1, U$3.GND, VR1.GND
- net N$14: now also C8.+, L1.2, R4.2; no longer CHRGNG.C, R6.1
- net N$2: now also BT1.+, BT2.-; no longer D1.A, L1.2, VR1.SW
- net N$3: now also L1.1, VR1.OUTPUT; no longer R3.1
Other:
- note removed: "Charging Circuit"
- moved on the sheet: BT1, C12, C9, L1, POWER_SWITCH, R3, R4, VR1
